File: Snugon_MO1_PCB/chip_sencor2 No2_back/Chip_Sencor2.kicad_sch (KiCad schematic)
At the start: 6 parts, among them J2 Conn_01x8_Pin + 2, SW10 SW_PUSH, SW11 SW_PUSH, SW7 SW_PUSH, SW8 SW_PUSH, SW9 SW_PUSH

Commit message: スイッチとエンコーダーはPCBAしない
Parts:
- SW10, SW11, SW7, SW8, SW9: LCSC C400268 -> (none)
Changed lines of the file:
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@@
       (effects (font (size 1.27 1.27)))
     )
-    (property "LCSC" "C400268" (at 158.75 90.17 0)
+    (property "LCSC" "" (at 158.75 90.17 0)
       (effects (font (size 1.27 1.27)) hide)
     )
@@
       (effects (font (size 1.27 1.27)))
     )
-    (property "LCSC" "C400268" (at 158.75 74.93 0)
+    (property "LCSC" "" (at 158.75 74.93 0)
       (effects (font (size 1.27 1.27)) hide)
     )
@@
       (effects (font (size 1.27 1.27)))
     )
-    (property "LCSC" "C400268" (at 158.75 59.69 0)
+    (property "LCSC" "" (at 158.75 59.69 0)
       (effects (font (size 1.27 1.27)) hide)
     )
@@
       (effects (font (size 1.27 1.27)))
     )
-    (property "LCSC" "C400268" (at 158.75 105.41 0)
+    (property "LCSC" "" (at 158.75 105.41 0)
       (effects (font (size 1.27 1.27)) hide)
     )
@@
       (effects (font (size 1.27 1.27)))
     )
-    (property "LCSC" "C400268" (at 158.75 120.65 0)
-      (effects (font (size 1.27 1.27)) hide)
-    )
+    (property "LCSC" "" (at 158.75 120.65 0)
+      (effects (font (size 1.27 1.27)) hide)
+    )
