File: Snugon_MO1_PCB/chip_sencor2 No2_main/Sensor.kicad_sch (KiCad schematic)
At the start: 17 parts, among them U2 TPS73601DBV, U3 TXS0102DCU, U4 TXS0102DCU, U5 PMW3360DM-T2QU

Commit message: スイッチとエンコーダーはPCBAしない
Parts:
- U5: LCSC C20612443 -> (none)
Changed lines of the file:
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@@
       (effects (font (size 1.27 1.27)) (justify bottom) hide)
     )
-    (property "LCSC" "C20612443" (at 210.82 86.36 0)
+    (property "LCSC" "" (at 210.82 86.36 0)
       (effects (font (size 1.27 1.27)) hide)
     )
